File: kicad/power_board/power_board.kicad_pcb (KiCad board)
At the start: 2 copper layers, 99.1 x 99.1 mm, 37 parts, among them J1 multi_plexor_extra, J10 5V, J11 5V, J18 11.1V, J19 11.1V, J2 PowerInput, J20 11.1V, J21 11.1V, J22 11.1V, J23 11.1V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

Commit message: updated power board
Connections:
- sensor_7 pad 2: Net-(sensor_7-Pad2) -> GND
Changed lines of the file:
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@@
-(kicad_pcb (version 20171130) (host pcbnew "(5.1.6)-1")
+(kicad_pcb (version 20171130) (host pcbnew 5.1.5+dfsg1-2build2)
   (general
     (thickness 1.6)
@@
     (zones 0)
     (modules 37)
-    (nets 54)
+    (nets 53)
   )
   (page A4)
@@
   )
   (setup
-    (last_trace_width 1)
+    (last_trace_width 0.25)
     (user_trace_width 1)
     (user_trace_width 2)
@@
   (net 51 SDA7)
   (net 52 SCL7)
-  (net 53 "Net-(sensor_7-Pad2)")
   (net_class Default "This is the default net class."
     (clearance 0.2)
@@
     (add_net "Net-(D1-Pad1)")
     (add_net "Net-(R2-Pad2)")
-    (add_net "Net-(sensor_7-Pad2)")
     (add_net RESET_28)
     (add_net RESET_3)
@@
       (net 50 SDA6))
     (pad 2 thru_hole circle (at 2.54 0 180) (size 1.524 1.524) (drill 0.762) (layers *.Cu *.Mask)
-      (net 53 "Net-(sensor_7-Pad2)"))
+      (net 7 GND))
     (pad 1 thru_hole circle (at 0 0 180) (size 1.524 1.524) (drill 0.762) (layers *.Cu *.Mask)
       (net 30 +5V))
@@
   (module mercury:proto (layer F.Cu)
     (at 212.09 87.63 90)
-    (fp_text reference U3 (at 0 0.5 90) (layer F.SilkS)
-      (effects (font (size 1 1) (thickness 0.15)))
-    )
-    (fp_text value proto (at 0 -0.5 90) (layer F.Fab)
-      (effects (font (size 1 1) (thickness 0.15)))
-    )
-    (fp_text user REF** (at 0 -14.74 90) (layer F.SilkS)
-      (effects (font (size 1 1) (thickness 0.15)))
-    )
-    (fp_text user proto (at 0 -15.74 90) (layer F.Fab)
-      (effects (font (size 1 1) (thickness 0.15)))
-    )
-    (fp_text user REF** (at 0 -12.2 90) (layer F.SilkS)
-      (effects (font (size 1 1) (thickness 0.15)))
-    )
-    (fp_text user proto (at 0 -13.2 90) (layer F.Fab)
-      (effects (font (size 1 1) (thickness 0.15)))
-    )
-    (fp_text user REF** (at 0 -9.66 90) (layer F.SilkS)
-      (effects (font (size 1 1) (thickness 0.15)))
-    )
-    (fp_text user proto (at 0 -10.66 90) (layer F.Fab)
-      (effects (font (size 1 1) (thickness 0.15)))
-    )
-    (fp_text user REF** (at 0 -7.12 90) (layer F.SilkS)
-      (effects (font (size 1 1) (thickness 0.15)))
-    )
-    (fp_text user proto (at 0 -8.12 90) (layer F.Fab)
-      (effects (font (size 1 1) (thickness 0.15)))
-    )
-    (fp_text user REF** (at 0 -4.58 90) (layer F.SilkS)
-      (effects (font (size 1 1) (thickness 0.15)))
-    )
-    (fp_text user proto (at 0 -5.58 90) (layer F.Fab)
-      (effects (font (size 1 1) (thickness 0.15)))
-    )
-    (fp_text user REF** (at 0 -2.04 90) (layer F.SilkS)
-      (effects (font (size 1 1) (thickness 0.15)))
-    )
-    (fp_text user proto (at 0 -3.04 90) (layer F.Fab)
-      (effects (font (size 1 1) (thickness 0.15)))
-    )
+    (fp_text reference U3 (at 0 2.54 90) (layer F.SilkS)
+      (effects (font (size 1 1) (thickness 0.15)))
+    )
+    (fp_text value proto (at -3.81 -0.5 90) (layer F.Fab)
+      (effects (font (size 1 1) (thickness 0.15)))
+    )
+    (fp_text user proto (at -2.54 -15.24 90) (layer F.Fab)
+      (effects (font (size 1 1) (thickness 0.15)))
+    )
+    (fp_text user proto (at -2.54 -13.2 90) (layer F.Fab)
+      (effects (font (size 1 1) (thickness 0.15)))
+    )
+    (fp_text user proto (at -2.54 -11.43 90) (layer F.Fab)
+      (effects (font (size 1 1) (thickness 0.15)))
+    )
+    (fp_text user proto (at -3.81 -7.62 90) (layer F.Fab)
+      (effects (font (size 1 1) (thickness 0.15)))
+    )
+    (fp_text user proto (at -3.81 -5.58 90) (layer F.Fab)
+      (effects (font (size 1 1) (thickness 0.15)))
+    )
+    (fp_text user proto (at -3.81 -3.04 90) (layer F.Fab)
+      (effects (font (size 1 1) (thickness 0.15)))
+    )
