File: kicad/power_board/power_board.sch (KiCad schematic (older format))
At the start: 37 parts, among them J1 multi_plexor_extra, J10 5V, J11 5V, J18 11.1V, J19 11.1V, J2 PowerInput, J20 11.1V, J21 11.1V, J22 11.1V, J23 11.1V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

Commit message: updated power board
Parts:
- removed R2: 121Ohm, Resistor_THT:R_Axial_DIN0204_L3.6mm_D1.6mm_P7.62mm_Horizontal, symbol Device:R
- removed R3: 365Ohm, Resistor_THT:R_Axial_DIN0204_L3.6mm_D1.6mm_P7.62mm_Horizontal, symbol Device:R
- added J12: Raspberry_Pi_2_3, symbol Connector:Raspberry_Pi_2_3
- added U4: PCA9685, symbol mercury:PCA9685
- added ULeft1, URight1: motor_driver, symbol mercury:motor_driver
- D1: symbol dk_LED-Indication-Discrete:LTL2R3KGKNN -> power_board-rescue:LTL2R3KGKNN-dk_LED-Indication-Discrete
Connections:
- net labels added: GPIO12, GPIO13, GPIO18, GPIO19, GPIO20, GPIO21, GPIO5, GPIO6, ServoPWMSCL, ServoPWSDA
- no-connect marks 0 -> 1
Other:
- moved on the sheet: J1, U1
