File: kicad/Mercury 2021/Mercury 2021.kicad_pcb (KiCad board)
At the start: 2 copper layers, 100 x 100 mm, 46 parts, among them J1 Batt_Power, J10 3.3v rail, J13 Screw_Terminal_01x02, J14 Screw_Terminal_01x02, J15 Raspberry_Pi_2_3, J16 Sensors_Extra, J17 Arduino_Extra_Power, J18 Arduino_Extra_Comm, J19 Arduino_Extra_Digital, J2 Conn_01x20_Female, J20 Arduino_Extra_Analog, J21 MP_Extra_Analog, J3 Conn_01x20_Female, J30 Screw_Terminal_01x02, J31 Screw_Terminal_01x02, J32 Screw_Terminal_01x02, J33 Screw_Terminal_01x02, J36 GND rail 2, J37 GND rail 3, J4 Screw_Terminal_01x02, J5 Screw_Terminal_01x02, J7 5V rail, J8 GND Rail 1, J9 11v rail, U1 LM1084-5.0, U10 TCA9548APWR, U11 MDD10A, U12 PCA9685, U12C1 PCA9685, U13 MDD10A, U2 Adafruit_VL53L0X, U3 Adafruit_VL53L0X, U4 Adafruit_VL53L0X, U5 Adafruit_VL53L0X, U6 Adafruit_VL53L0X, U7 Adafruit_VL53L0X, U8 Adafruit_VL53L0X, U9 Adafruit_VL53L0X

Commit message: Ordered the pcb
Parts:
- moved U12 38.3 mm to (106.7, 77.5)
Routing:
- net /Motors/Pi03: track 32.3 -> 75.9 mm
- net /Motors/Pi05: track 37.4 -> 79.2 mm
- net /Motors/Pi14: track 36.0 -> 77.5 mm
Other:
- board text added: "Board by: Max Myzer With contributions from: c3n3"
- board text removed: "Board by: Max Myzer With contributions from: CNC3"
